Commit message: 20220128-1

File: hrwros_support/urdf/turtlebot3_with_carrier/turtlebot3_waffle_with_carrier.urdf.xacro (robot description, xacro)
@@ -19,5 +19,5 @@
       <color rgba="0.7 0.7 0.7 1.0" />
   </material>
-  <xacro:include filename="$(find turtlebot3_description)/urdf/turtlebot3_waffle.urdf.xacro"/>
+  <xacro:include filename="$(find turtlebot3_description)/urdf/turtlebot3_waffle_pi.urdf.xacro"/>
   <link name="carrierplate_link">
     <visual>
@@ -29,6 +29,6 @@
     </visual>
     <inertial>
-      <mass value="0.1"/>
-      <xacro:box_inertia m="0.1" x="0.26" y="0.26" z="0.008"/>
+      <mass value="0.001"/>
+      <xacro:box_inertia m="0.001" x="0.26" y="0.26" z="0.008"/>
     </inertial>
     <collision>
@@ -37,4 +37,12 @@
         <box size="0.26 0.26 0.008"/>
       </geometry>
+      <surface>
+        <friction>
+          <ode>
+            <mu>0.5</mu>
+            <mu2>0.5</mu2>
+          </ode>
+        </friction>
+      </surface>
    </collision>
   </link>

Commit message: 20220128-5

File: hrwros_support/urdf/turtlebot3_with_carrier/turtlebot3_waffle_with_carrier.urdf.xacro (robot description, xacro)
@@ -22,7 +22,7 @@
   <link name="carrierplate_link">
     <visual>
-      <origin xyz="-0.06 0.0 0.0" />
+      <origin xyz="0.0 0.0 0.0" />
       <geometry>
-        <box size="0.26 0.26 0.008" />
+        <box size="0.36 0.36 0.008" />
       </geometry>
       <material name="LightGrey"/>
@@ -30,16 +30,16 @@
     <inertial>
       <mass value="0.001"/>
-      <xacro:box_inertia m="0.001" x="0.26" y="0.26" z="0.008"/>
+      <xacro:box_inertia m="0.001" x="0.36" y="0.36" z="0.008"/>
     </inertial>
     <collision>
       <origin xyz="0 0 0" rpy="0 0 0"/>
       <geometry>
-        <box size="0.26 0.26 0.008"/>
+        <box size="0.36 0.36 0.008"/>
       </geometry>
       <surface>
         <friction>
           <ode>
-            <mu>0.5</mu>
-            <mu2>0.5</mu2>
+            <mu>10</mu>
+            <mu2>10</mu2>
           </ode>
         </friction>
@@ -47,6 +47,134 @@
    </collision>
   </link>
+  <link name="randje1_link">
+    <visual>
+      <origin xyz="0.0 0.0 0.0" />
+      <geometry>
+        <box size="0.36 0.01 0.01" />
+      </geometry>
+      <material name="LightGrey"/>
+    </visual>
+    <inertial>
+      <mass value="0.0001"/>
+      <xacro:box_inertia m="0.0001" x="0.36" y="0.001" z="0.001"/>
+    </inertial>
+    <collision>
+      <origin xyz="0 0 0" rpy="0 0 0"/>
+      <geometry>
+        <box size="0.36 0.01 0.01"/>
+      </geometry>
+      <surface>
+        <friction>
+          <ode>
+            <mu>10</mu>
+            <mu2>10</mu2>
+          </ode>
+        </friction>
+      </surface>
+   </collision>
+  </link>
+  <link name="randje2_link">
+    <visual>
+      <origin xyz="0.0 0.0 0.0" />
+      <geometry>
+        <box size="0.36 0.01 0.01" />
+      </geometry>
+      <material name="LightGrey"/>
+    </visual>
+    <inertial>
+      <mass value="0.0001"/>
+      <xacro:box_inertia m="0.0001" x="0.36" y="0.001" z="0.001"/>
+    </inertial>
+    <collision>
+      <origin xyz="0 0 0" rpy="0 0 0"/>
+      <geometry>
+        <box size="0.36 0.01 0.01"/>
+      </geometry>
+      <surface>
+        <friction>
+          <ode>
+            <mu>10</mu>
+            <mu2>10</mu2>
+          </ode>
+        </friction>
+      </surface>
+   </collision>
+  </link>
+  <link name="randje3_link">
+    <visual>
+      <origin xyz="0.0 0.0 0.0" />
+      <geometry>
+        <box size="0.36 0.01 0.01" />
+      </geometry>
+      <material name="LightGrey"/>
+    </visual>
+    <inertial>
+      <mass value="0.0001"/>
+      <xacro:box_inertia m="0.0001" x="0.36" y="0.001" z="0.001"/>
+    </inertial>
+    <collision>
+      <origin xyz="0 0 0" rpy="0 0 0"/>
+      <geometry>
+        <box size="0.36 0.01 0.01"/>
+      </geometry>
+      <surface>
+        <friction>
+          <ode>
+            <mu>10</mu>
+            <mu2>10</mu2>
+          </ode>
+        </friction>
+      </surface>
+   </collision>
+  </link>
+  <link name="randje4_link">
+    <visual>
+      <origin xyz="0.0 0.0 0.0" />
+      <geometry>
+        <box size="0.36 0.01 0.01" />
+      </geometry>
+      <material name="LightGrey"/>
+    </visual>
+    <inertial>
+      <mass value="0.0001"/>
+      <xacro:box_inertia m="0.0001" x="0.36" y="0.001" z="0.001"/>
+    </inertial>
+    <collision>
+      <origin xyz="0 0 0" rpy="0 0 0"/>
+      <geometry>
+        <box size="0.36 0.01 0.01"/>
+      </geometry>
+      <surface>
+        <friction>
+          <ode>
+            <mu>10</mu>
+            <mu2>10</mu2>
+          </ode>
+        </friction>
+      </surface>
+   </collision>
+  </link>
+  <joint name="randje1_jount" type="fixed">
+    <origin xyz="0.18 0 0.008" rpy="0.0 0.0 ${pi/2}"/>
+    <parent link="carrierplate_link" />
+    <child link="randje1_link" />
+  </joint>
+  <joint name="randje2_jount" type="fixed">
+    <origin xyz="-0.18 0 0.008" rpy="0.0 0.0 ${pi/2}"/>
+    <parent link="carrierplate_link" />
+    <child link="randje2_link" />
+  </joint>
+  <joint name="randje3_jount" type="fixed">
+    <origin xyz="0.0 0.18 0.008" rpy="0.0 0.0 0.0"/>
+    <parent link="carrierplate_link" />
+    <child link="randje3_link" />
+  </joint>
+  <joint name="randje4_jount" type="fixed">
+    <origin xyz="0.0 -0.18 0.008" rpy="0.0 0.0 0.0"/>
+    <parent link="carrierplate_link" />
+    <child link="randje4_link" />
+  </joint>
   <joint name="carrierplate_joint" type="fixed">
-    <origin xyz="0.0 0 0.4" rpy="0.0 0.0 0.0"/>
+    <origin xyz="-0.06 0 0.4" rpy="0.0 0.0 0.0"/>
     <parent link="base_link" />
     <child link="carrierplate_link" />

Commit message: 20220130

File: hrwros_support/urdf/turtlebot3_with_carrier/turtlebot3_waffle_with_carrier.urdf.xacro (robot description, xacro)
@@ -1,178 +1,6 @@
 <?xml version="1.0" ?>
 <robot name="turtlebot3_waffle_with_carrier" xmlns:xacro="http://ros.org/wiki/xacro">
-  <xacro:macro name="cylinder_inertia" params="m r h">
-        <inertia  ixx="${m*(3*r*r+h*h)/12}" ixy = "0" ixz = "0"
-                    iyy="${m*(3*r*r+h*h)/12}" iyz = "0"
-                    izz="${m*r*r/2}" />
-  </xacro:macro>
-  <xacro:macro name="box_inertia" params="m x y z">
-          <inertia  ixx="${m*(y*y+z*z)/12}" ixy = "0" ixz = "0"
-                    iyy="${m*(x*x+z*z)/12}" iyz = "0"
-                    izz="${m*(x*x+z*z)/12}" />
-  </xacro:macro>
-  <xacro:macro name="sphere_inertia" params="m r">
-          <inertia  ixx="${2*m*r*r/5}" ixy = "0" ixz = "0"
-                    iyy="${2*m*r*r/5}" iyz = "0"
-                    izz="${2*m*r*r/5}" />
-  </xacro:macro>
-  <material name="LightGrey">
-      <color rgba="0.7 0.7 0.7 1.0" />
-  </material>
   <xacro:include filename="$(find turtlebot3_description)/urdf/turtlebot3_waffle_pi.urdf.xacro"/>
-  <link name="carrierplate_link">
-    <visual>
-      <origin xyz="0.0 0.0 0.0" />
-      <geometry>
-        <box size="0.36 0.36 0.008" />
-      </geometry>
-      <material name="LightGrey"/>
-    </visual>
-    <inertial>
-      <mass value="0.001"/>
-      <xacro:box_inertia m="0.001" x="0.36" y="0.36" z="0.008"/>
-    </inertial>
-    <collision>
-      <origin xyz="0 0 0" rpy="0 0 0"/>
-      <geometry>
-        <box size="0.36 0.36 0.008"/>
-      </geometry>
-      <surface>
-        <friction>
-          <ode>
-            <mu>10</mu>
-            <mu2>10</mu2>
-          </ode>
-        </friction>
-      </surface>
-   </collision>
-  </link>
-  <link name="randje1_link">
-    <visual>
-      <origin xyz="0.0 0.0 0.0" />
-      <geometry>
-        <box size="0.36 0.01 0.01" />
-      </geometry>
-      <material name="LightGrey"/>
-    </visual>
-    <inertial>
-      <mass value="0.0001"/>
-      <xacro:box_inertia m="0.0001" x="0.36" y="0.001" z="0.001"/>
-    </inertial>
-    <collision>
-      <origin xyz="0 0 0" rpy="0 0 0"/>
-      <geometry>
-        <box size="0.36 0.01 0.01"/>
-      </geometry>
-      <surface>
-        <friction>
-          <ode>
-            <mu>10</mu>
-            <mu2>10</mu2>
-          </ode>
-        </friction>
-      </surface>
-   </collision>
-  </link>
-  <link name="randje2_link">
-    <visual>
-      <origin xyz="0.0 0.0 0.0" />
-      <geometry>
-        <box size="0.36 0.01 0.01" />
-      </geometry>
-      <material name="LightGrey"/>
-    </visual>
-    <inertial>
-      <mass value="0.0001"/>
-      <xacro:box_inertia m="0.0001" x="0.36" y="0.001" z="0.001"/>
-    </inertial>
-    <collision>
-      <origin xyz="0 0 0" rpy="0 0 0"/>
-      <geometry>
-        <box size="0.36 0.01 0.01"/>
-      </geometry>
-      <surface>
-        <friction>
-          <ode>
-            <mu>10</mu>
-            <mu2>10</mu2>
-          </ode>
-        </friction>
-      </surface>
-   </collision>
-  </link>
-  <link name="randje3_link">
-    <visual>
-      <origin xyz="0.0 0.0 0.0" />
-      <geometry>
-        <box size="0.36 0.01 0.01" />
-      </geometry>
-      <material name="LightGrey"/>
-    </visual>
-    <inertial>
-      <mass value="0.0001"/>
-      <xacro:box_inertia m="0.0001" x="0.36" y="0.001" z="0.001"/>
-    </inertial>
-    <collision>
-      <origin xyz="0 0 0" rpy="0 0 0"/>
-      <geometry>
-        <box size="0.36 0.01 0.01"/>
-      </geometry>
-      <surface>
-        <friction>
-          <ode>
-            <mu>10</mu>
-            <mu2>10</mu2>
-          </ode>
-        </friction>
-      </surface>
-   </collision>
-  </link>
-  <link name="randje4_link">
-    <visual>
-      <origin xyz="0.0 0.0 0.0" />
-      <geometry>
-        <box size="0.36 0.01 0.01" />
-      </geometry>
-      <material name="LightGrey"/>
-    </visual>
-    <inertial>
-      <mass value="0.0001"/>
-      <xacro:box_inertia m="0.0001" x="0.36" y="0.001" z="0.001"/>
-    </inertial>
-    <collision>
-      <origin xyz="0 0 0" rpy="0 0 0"/>
-      <geometry>
-        <box size="0.36 0.01 0.01"/>
-      </geometry>
-      <surface>
-        <friction>
-          <ode>
-            <mu>10</mu>
-            <mu2>10</mu2>
-          </ode>
-        </friction>
-      </surface>
-   </collision>
-  </link>
-  <joint name="randje1_jount" type="fixed">
-    <origin xyz="0.18 0 0.008" rpy="0.0 0.0 ${pi/2}"/>
-    <parent link="carrierplate_link" />
-    <child link="randje1_link" />
-  </joint>
-  <joint name="randje2_jount" type="fixed">
-    <origin xyz="-0.18 0 0.008" rpy="0.0 0.0 ${pi/2}"/>
-    <parent link="carrierplate_link" />
-    <child link="randje2_link" />
-  </joint>
-  <joint name="randje3_jount" type="fixed">
-    <origin xyz="0.0 0.18 0.008" rpy="0.0 0.0 0.0"/>
-    <parent link="carrierplate_link" />
-    <child link="randje3_link" />
-  </joint>
-  <joint name="randje4_jount" type="fixed">
-    <origin xyz="0.0 -0.18 0.008" rpy="0.0 0.0 0.0"/>
-    <parent link="carrierplate_link" />
-    <child link="randje4_link" />
-  </joint>
+  <xacro:include filename="$(find hrwros_support)/urdf/turtlebot3_with_carrier/turtlebot3_carrier.urdf.xacro"/>
   <joint name="carrierplate_joint" type="fixed">
     <origin xyz="-0.06 0 0.4" rpy="0.0 0.0 0.0"/>
